File: ilulissat.sch (KiCad schematic (older format))
At the start: 26 parts, among them J1 Conn_01x04, U1 EFR32MG21x, U2 HDC2080, Y1 32678Hz, Y2 28.4Mhz

Commit message: Start adding footprints, fill in remaining components
Parts:
- removed J1: Conn_01x04, symbol Connector_Generic:Conn_01x04
- added BT1: Battery_Cell, symbol Device:Battery_Cell
- added J1: Conn_01x02, symbol Connector_Generic:Conn_01x02
- added SW1: SW_SPST, Button_Switch_SMD:SW_SPST_B3U-1000P, symbol Switch:SW_SPST
- AE1: LCSC (none) -> C127620
- C1, C10, C11, C12, C13, C14, C15, C2, C3, C4, C5, C6, C7, C8, C9: footprint (none) -> Capacitor_SMD:C_0402_1005Metric
- R1, R2: value R_Small -> 100k; footprint (none) -> Resistor_SMD:R_0402_1005Metric
- U1: footprint (none) -> Package_DFN_QFN:QFN-32-1EP_4x4mm_P0.4mm_EP2.65x2.65mm
- Y1: value 32678Hz -> 32.768Khz; footprint (none) -> Crystal:Crystal_SMD_3215-2Pin_3.2x1.5mm; LCSC (none) -> C390740
- Y2: value 28.4Mhz -> 38.4Mhz; footprint (none) -> Crystal:Crystal_SMD_2520-4Pin_2.5x2.0mm; LCSC (none) -> C409422
Connections:
- net labels added: ANT-, HDC_INT, HDC_SCL, HDC_SDA, ~RESET~
- net labels removed: INT, SCL, SDA
- wire segments 109 -> 115
- no-connect marks 1 -> 15

Commit message: More parts
Parts:
- AE1: footprint (none) -> Antenna_Extra:2450AT18A100
- BT1: value Battery_Cell -> CR2032; footprint (none) -> batt:BAT-HLD-001-THM
- L1, L2: footprint (none) -> Inductor_SMD:L_0402_1005Metric; LCSC (none) -> C281011
- L3: footprint (none) -> Inductor_SMD:L_0402_1005Metric
Connections:
- net labels added: ANT+
Other:
- moved on the sheet: AE1
Changed lines of the file:
@@
 F 0 "L1" H 2400 2200 50  0000 L CNN
 F 1 "9.1nH" V 2600 2200 50  0000 L CNN
-F 2 "" H 2500 2250 50  0001 C CNN
-F 3 "~" H 2500 2250 50  0001 C CNN
+F 2 "Inductor_SMD:L_0402_1005Metric" H 2500 2250 50  0001 C CNN
+F 3 "https://datasheet.lcsc.com/szlcsc/1811141856_microgate-MGCI1005T9N1ST-LF_C281011.pdf" H 2500 2250 50  0001 C CNN
+F 4 "C281011" H 2500 2250 50  0001 C CNN "LCSC"
 	1    2500 2250
 	1    0    0    -1
@@
 F 0 "L2" H 2650 2200 50  0000 L CNN
 F 1 "9.1nH" V 2800 2200 50  0000 L CNN
-F 2 "" H 2750 2250 50  0001 C CNN
-F 3 "~" H 2750 2250 50  0001 C CNN
+F 2 "Inductor_SMD:L_0402_1005Metric" H 2750 2250 50  0001 C CNN
+F 3 "https://datasheet.lcsc.com/szlcsc/1811141856_microgate-MGCI1005T9N1ST-LF_C281011.pdf" H 2750 2250 50  0001 C CNN
+F 4 "C281011" H 2750 2250 50  0001 C CNN "LCSC"
 	1    2750 2250
 	1    0    0    -1
@@
 F 0 "L3" V 4785 3900 50  0000 C CNN
 F 1 "2.0nH" V 4694 3900 50  0000 C CNN
-F 2 "" H 4600 3900 50  0001 C CNN
+F 2 "Inductor_SMD:L_0402_1005Metric" H 4600 3900 50  0001 C CNN
 F 3 "~" H 4600 3900 50  0001 C CNN
 	1    4600 3900
@@
 L Device:Antenna_Chip AE1
 U 1 1 5E29AE31
-P 5850 3800
-F 0 "AE1" V 5822 4104 50  0000 L CNN
-F 1 "Antenna_Chip" V 5913 4104 50  0000 L CNN
-F 2 "" H 5750 3975 50  0001 C CNN
-F 3 "https://datasheet.lcsc.com/szlcsc/1808272258_Walsin-Tech-Corp-RFECA3216060A1T_C127620.pdf" H 5750 3975 50  0001 C CNN
-F 4 "C127620" H 5850 3800 50  0001 C CNN "LCSC"
-	1    5850 3800
+P 5850 4000
+F 0 "AE1" V 5822 4304 50  0000 L CNN
+F 1 "Antenna_Chip" V 5913 4304 50  0000 L CNN
+F 2 "Antenna_Extra:2450AT18A100" H 5750 4175 50  0001 C CNN
+F 3 "https://datasheet.lcsc.com/szlcsc/1808272258_Walsin-Tech-Corp-RFECA3216060A1T_C127620.pdf" H 5750 4175 50  0001 C CNN
+F 4 "C127620" H 5850 4000 50  0001 C CNN "LCSC"
+	1    5850 4000
 	0    1    1    0
 $EndComp
@@
 	1950 4100 1950 4050
 Text Label 3700 3900 0    50   ~ 0
-ANT-
+ANT+
 Text Label 3700 4000 0    50   ~ 0
 ANT-
@@
 P 1000 1850
 F 0 "BT1" H 1118 1946 50  0000 L CNN
-F 1 "Battery_Cell" H 1118 1855 50  0000 L CNN
-F 2 "" V 1000 1910 50  0001 C CNN
+F 1 "CR2032" H 1118 1855 50  0000 L CNN
+F 2 "batt:BAT-HLD-001-THM" V 1000 1910 50  0001 C CNN
 F 3 "~" V 1000 1910 50  0001 C CNN
 	1    1000 1850
@@
 Wire Wire Line
 	1000 1550 1000 1650
-NoConn ~ 5750 3700
+NoConn ~ 5750 4100
 Text Label 9700 2200 0    50   ~ 0
 SWDIO
@@
 F 1 "Conn_01x02" H 10530 2101 50  0000 L CNN
 F 2 "" H 10450 2200 50  0001 C CNN
-F 3 "~" H 10450 2200 50  0001 C CNN
+F 3 "" H 10450 2200 50  0001 C CNN
 	1    10450 2200
 	1    0    0    -1

Commit message: WIP WIP
Parts:
- removed J1: Conn_01x02, symbol Connector_Generic:Conn_01x02
- added L4: 0R, Inductor_SMD:L_0402_1005Metric, symbol Device:L_Small
- added TP101: SWDIO, TestPoint:TestPoint_Pad_D1.0mm, symbol Connector:TestPoint
- added TP102: SWCLK, TestPoint:TestPoint_Pad_D1.0mm, symbol Connector:TestPoint
- AE1: footprint Antenna_Extra:2450AT18A100 -> Antenna_Extra:Antenna_Johanson_2450AT42E0100
- BT1: footprint batt:BAT-HLD-001-THM -> batt:BatteryHolder_Linx_BAT-HLD-001-THM
- Y1: footprint Crystal:Crystal_SMD_3215-2Pin_3.2x1.5mm -> Crystal:Crystal_SMD_2012-2Pin_2.0x1.2mm
- Y2: footprint Crystal:Crystal_SMD_2520-4Pin_2.5x2.0mm -> Crystal:Crystal_SMD_2016-4Pin_2.0x1.6mm
Connections:
- net labels added: +, -, HFXTAL_I, HFXTAL_O, LFXTAL_I, LFXTAL_O, PAVDD, RFVDD
- wire segments 115 -> 118
- no-connect marks 15 -> 14
Other:
- moved on the sheet: AE1
Changed lines of the file:
@@
 L Device:Antenna_Chip AE1
 U 1 1 5E29AE31
-P 5850 4000
-F 0 "AE1" V 5822 4304 50  0000 L CNN
-F 1 "Antenna_Chip" V 5913 4304 50  0000 L CNN
-F 2 "Antenna_Extra:2450AT18A100" H 5750 4175 50  0001 C CNN
-F 3 "https://datasheet.lcsc.com/szlcsc/1808272258_Walsin-Tech-Corp-RFECA3216060A1T_C127620.pdf" H 5750 4175 50  0001 C CNN
-F 4 "C127620" H 5850 4000 50  0001 C CNN "LCSC"
-	1    5850 4000
-	0    1    1    0
-$EndComp
-Wire Wire Line
-	5750 3900 5400 3900
+P 6150 3500
+F 0 "AE1" V 6122 3804 50  0000 L CNN
+F 1 "Antenna_Chip" V 6213 3804 50  0000 L CNN
+F 2 "Antenna_Extra:Antenna_Johanson_2450AT42E0100" H 6050 3675 50  0001 C CNN
+F 3 "https://datasheet.lcsc.com/szlcsc/1808272258_Walsin-Tech-Corp-RFECA3216060A1T_C127620.pdf" H 6050 3675 50  0001 C CNN
+F 4 "C127620" H 6150 3500 50  0001 C CNN "LCSC"
+	1    6150 3500
+	-1   0    0    -1
+$EndComp
 $Comp
 L Device:Crystal_Small Y1
@@
 F 0 "Y1" V 1704 3938 50  0000 L CNN
 F 1 "32.768Khz" V 1795 3938 50  0000 L CNN
-F 2 "Crystal:Crystal_SMD_3215-2Pin_3.2x1.5mm" H 1750 3850 50  0001 C CNN
+F 2 "Crystal:Crystal_SMD_2012-2Pin_2.0x1.2mm" H 1750 3850 50  0001 C CNN
 F 3 "https://datasheet.lcsc.com/szlcsc/1912111437_JGHC-SMD31327681252090_C390740.pdf" H 1750 3850 50  0001 C CNN
 F 4 "C390740" H 1750 3850 50  0001 C CNN "LCSC"
@@
 F 0 "Y2" V 1500 4000 50  0000 L CNN
 F 1 "38.4Mhz" V 1800 4050 50  0000 L CNN
-F 2 "Crystal:Crystal_SMD_2520-4Pin_2.5x2.0mm" H 1600 4150 50  0001 C CNN
+F 2 "Crystal:Crystal_SMD_2016-4Pin_2.0x1.6mm" H 1600 4150 50  0001 C CNN
 F 3 "https://datasheet.lcsc.com/szlcsc/1912111437_KYX-K2C384001010_C409422.pdf" H 1600 4150 50  0001 C CNN
 F 4 "C409422" V 1600 4150 50  0001 C CNN "LCSC"
@@
 Text Label 5500 2050 0    50   ~ 0
 HDC_INT
-Wire Wire Line
-	10250 2200 9500 2200
 Wire Wire Line
 	10250 2300 9500 2300
@@
 F 0 "BT1" H 1118 1946 50  0000 L CNN
 F 1 "CR2032" H 1118 1855 50  0000 L CNN
-F 2 "batt:BAT-HLD-001-THM" V 1000 1910 50  0001 C CNN
+F 2 "batt:BatteryHolder_Linx_BAT-HLD-001-THM" V 1000 1910 50  0001 C CNN
 F 3 "~" V 1000 1910 50  0001 C CNN
 	1    1000 1850
@@
 Wire Wire Line
 	1000 1550 1000 1650
-NoConn ~ 5750 4100
 Text Label 9700 2200 0    50   ~ 0
 SWDIO
 Text Label 9700 2300 0    50   ~ 0
 SWCLK
-$Comp
-L Connector_Generic:Conn_01x02 J1
-U 1 1 5E35DD5F
-P 10450 2200
-F 0 "J1" H 10530 2192 50  0000 L CNN
-F 1 "Conn_01x02" H 10530 2101 50  0000 L CNN
-F 2 "" H 10450 2200 50  0001 C CNN
-F 3 "" H 10450 2200 50  0001 C CNN
-	1    10450 2200
-	1    0    0    -1
-$EndComp
 $Comp
 L Switch:SW_SPST SW1
@@
 	1000 2000 1000 2050
 Connection ~ 1000 2000
+Text Label 1000 1500 0    50   ~ 0
++
+Text Label 1000 1950 0    50   ~ 0
+-
+$Comp
+L Connector:TestPoint TP101
+U 1 1 5E38CEFE
+P 10250 2200
+F 0 "TP101" V 10055 2272 50  0000 C CNN
+F 1 "SWDIO" V 10146 2272 50  0000 C CNN
+F 2 "TestPoint:TestPoint_Pad_D1.0mm" H 10450 2200 50  0001 C CNN
+F 3 "~" H 10450 2200 50  0001 C CNN
+	1    10250 2200
+	0    1    1    0
+$EndComp
+$Comp
+L Connector:TestPoint TP102
+U 1 1 5E38D660
+P 10250 2300
+F 0 "TP102" V 10204 2488 50  0000 L CNN
+F 1 "SWCLK" V 10295 2488 50  0000 L CNN
+F 2 "TestPoint:TestPoint_Pad_D1.0mm" H 10450 2300 50  0001 C CNN
+F 3 "~" H 10450 2300 50  0001 C CNN
+	1    10250 2300
+	0    1    1    0
+$EndComp
+Wire Wire Line
+	10250 2200 9500 2200
+Text Label 2500 2400 1    50   ~ 0
+PAVDD
+Text Label 2750 2450 0    50   ~ 0
+RFVDD
+$Comp
+L power:GND #PWR0101
+U 1 1 5E3AE965
+P 6050 3650
+F 0 "#PWR0101" H 6050 3400 50  0001 C CNN
+F 1 "GND" H 6055 3477 50  0000 C CNN
+F 2 "" H 6050 3650 50  0001 C CNN
+F 3 "" H 6050 3650 50  0001 C CNN
+	1    6050 3650
+	1    0    0    -1
+$EndComp
+Wire Wire Line
+	6050 3600 6050 3650
+Wire Wire Line
+	6250 3900 6250 3600
+Wire Wire Line
+	5400 3900 5650 3900
+$Comp
+L Device:L_Small L4
+U 1 1 5E3D387B
+P 5750 3900
+F 0 "L4" V 5935 3900 50  0000 C CNN
+F 1 "0R" V 5844 3900 50  0000 C CNN
+F 2 "Inductor_SMD:L_0402_1005Metric" H 5750 3900 50  0001 C CNN
+F 3 "~" H 5750 3900 50  0001 C CNN
+	1    5750 3900
+	0    -1   -1   0
+$EndComp
+Wire Wire Line
+	5850 3900 6250 3900
+Text Label 1650 4050 0    50   ~ 0
+HFXTAL_I
+Text Label 1650 4250 0    50   ~ 0
+HFXTAL_O
+Text Label 1800 3750 0    50   ~ 0
+LFXTAL_I
+Text Label 1800 3950 0    50   ~ 0
+LFXTAL_O
 $EndSCHEMATC

Commit message: Routing complete, needs cleanup
Parts:
- removed C10: 10uF, Capacitor_SMD:C_0402_1005Metric, symbol Device:C_Small
- Y1: LCSC C390740 -> (none); Mouser (none) -> 520-.327-12.5-12R-T
- Y2: footprint Crystal:Crystal_SMD_2016-4Pin_2.0x1.6mm -> Crystal:Crystal_SMD_3225-4Pin_3.2x2.5mm; LCSC C409422 -> (none); Mouser (none) -> 520-384-10-33B-CKYT
Connections:
- wire segments 118 -> 114
Other:
- moved on the sheet: C11
Changed lines of the file:
@@
 $EndComp
 $Comp
-L Device:C_Small C10
-U 1 1 5E25275F
+L Device:C_Small C11
+U 1 1 5E252A4C
 P 2450 1050
-F 0 "C10" H 2358 1004 50  0000 R CNN
-F 1 "10uF" H 2358 1095 50  0000 R CNN
+F 0 "C11" H 2358 1004 50  0000 R CNN
+F 1 "10nF" H 2358 1095 50  0000 R CNN
 F 2 "Capacitor_SMD:C_0402_1005Metric" H 2450 1050 50  0001 C CNN
 F 3 "~" H 2450 1050 50  0001 C CNN
@@
 $EndComp
 $Comp
-L Device:C_Small C11
-U 1 1 5E252A4C
-P 2700 1050
-F 0 "C11" H 2608 1004 50  0000 R CNN
-F 1 "10nF" H 2608 1095 50  0000 R CNN
-F 2 "Capacitor_SMD:C_0402_1005Metric" H 2700 1050 50  0001 C CNN
-F 3 "~" H 2700 1050 50  0001 C CNN
-	1    2700 1050
-	-1   0    0    1
-$EndComp
-$Comp
 L power:GND #PWR02
 U 1 1 5E252EC8
-P 2700 1300
-F 0 "#PWR02" H 2700 1050 50  0001 C CNN
-F 1 "GND" H 2705 1127 50  0000 C CNN
-F 2 "" H 2700 1300 50  0001 C CNN
-F 3 "" H 2700 1300 50  0001 C CNN
-	1    2700 1300
+P 2450 1300
+F 0 "#PWR02" H 2450 1050 50  0001 C CNN
+F 1 "GND" H 2455 1127 50  0000 C CNN
+F 2 "" H 2450 1300 50  0001 C CNN
+F 3 "" H 2450 1300 50  0001 C CNN
+	1    2450 1300
 	1    0    0    -1
 $EndComp
@@
 	1550 1250 1800 1250
 Wire Wire Line
-	2700 1250 2700 1300
-Wire Wire Line
-	2700 1150 2700 1250
-Connection ~ 2700 1250
-Wire Wire Line
 	2450 1150 2450 1250
-Connection ~ 2450 1250
-Wire Wire Line
-	2450 1250 2700 1250
 Wire Wire Line
 	2250 1150 2250 1250
@@
 Wire Wire Line
 	1800 1250 2050 1250
-Wire Wire Line
-	2700 950  2700 850
-Wire Wire Line
-	2700 850  2450 850
 Connection ~ 1550 850
 Wire Wire Line
@@
 Wire Wire Line
 	2450 950  2450 850
-Connection ~ 2450 850
 Wire Wire Line
 	2450 850  2250 850
@@
 F 1 "32.768Khz" V 1795 3938 50  0000 L CNN
 F 2 "Crystal:Crystal_SMD_2012-2Pin_2.0x1.2mm" H 1750 3850 50  0001 C CNN
-F 3 "https://datasheet.lcsc.com/szlcsc/1912111437_JGHC-SMD31327681252090_C390740.pdf" H 1750 3850 50  0001 C CNN
-F 4 "C390740" H 1750 3850 50  0001 C CNN "LCSC"
+F 3 "https://www.mouser.dk/ProductDetail/ECS/ECS-327-125-12R-TR?qs=sGAEpiMZZMsBj6bBr9Q9abMK2mGYOCsJmFr8uZgFzeqFD0juhEFDSg==" H 1750 3850 50  0001 C CNN
+F 4 "520-.327-12.5-12R-T" V 1750 3850 50  0001 C CNN "Mouser"
 	1    1750 3850
 	0    1    1    0
@@
 F 0 "Y2" V 1500 4000 50  0000 L CNN
 F 1 "38.4Mhz" V 1800 4050 50  0000 L CNN
-F 2 "Crystal:Crystal_SMD_2016-4Pin_2.0x1.6mm" H 1600 4150 50  0001 C CNN
-F 3 "https://datasheet.lcsc.com/szlcsc/1912111437_KYX-K2C384001010_C409422.pdf" H 1600 4150 50  0001 C CNN
-F 4 "C409422" V 1600 4150 50  0001 C CNN "LCSC"
+F 2 "Crystal:Crystal_SMD_3225-4Pin_3.2x2.5mm" H 1600 4150 50  0001 C CNN
+F 3 "https://www.mouser.dk/ProductDetail/ECS/ECS-384-10-33B-CKY-TR?qs=sGAEpiMZZMsBj6bBr9Q9abMK2mGYOCsJg%2FKvxI2TTWJrWRS%252BDtNAig%3D%3D" H 1600 4150 50  0001 C CNN
+F 4 "520-384-10-33B-CKYT" V 1600 4150 50  0001 C CNN "Mouser"
 	1    1600 4150
 	0    1    1    0
@@
 ANT-
 Wire Wire Line
-	3650 2800 4050 2800
-Wire Wire Line
-	3650 2900 4050 2900
-Wire Wire Line
-	3650 3000 4050 3000
-Text Label 3700 2800 0    50   ~ 0
+	1750 3150 2150 3150
+Wire Wire Line
+	1750 3250 2150 3250
+Wire Wire Line
+	1750 3350 2150 3350
+Text Label 1800 3150 0    50   ~ 0
 HDC_SDA
-Text Label 3700 2900 0    50   ~ 0
+Text Label 1800 3350 0    50   ~ 0
 HDC_INT
-Text Label 3700 3000 0    50   ~ 0
+Text Label 1800 3250 0    50   ~ 0
 HDC_SCL
 NoConn ~ 3650 3100
@@
 NoConn ~ 3650 3300
 NoConn ~ 3650 3400
-NoConn ~ 2150 3150
-NoConn ~ 2150 3250
-NoConn ~ 2150 3350
 NoConn ~ 2150 3450
 NoConn ~ 2150 3550
@@
 Text Label 1800 3950 0    50   ~ 0
 LFXTAL_O
+Wire Wire Line
+	2450 1250 2450 1300
+Connection ~ 2450 1250
+NoConn ~ 3650 2800
+NoConn ~ 3650 2900
+NoConn ~ 3650 3000
 $EndSCHEMATC

Commit message: Add a user button
Parts:
- removed TP101: SWDIO, TestPoint:TestPoint_Pad_D1.0mm, symbol Connector:TestPoint
- removed TP102: SWCLK, TestPoint:TestPoint_Pad_D1.0mm, symbol Connector:TestPoint
- added J1: Conn_01x04, Connector_PinHeader_1.27mm:PinHeader_1x04_P1.27mm_Vertical, symbol Connector_Generic:Conn_01x04
- added SW2: USR, Button_Switch_SMD:SW_SPST_B3U-1000P, symbol Switch:SW_SPST
- SW1: value SW_SPST -> ~RST~
Connections:
- net labels added: ~USRBTN~
- wire segments 114 -> 119
- no-connect marks 14 -> 13
Changed lines of the file:
@@
 HDC_INT
 Wire Wire Line
-	10250 2300 9500 2300
+	10700 2300 9950 2300
 $Comp
 L power:GND #PWR015
@@
 NoConn ~ 3650 3300
 NoConn ~ 3650 3400
-NoConn ~ 2150 3450
 NoConn ~ 2150 3550
 NoConn ~ 2150 3650
@@
 Wire Wire Line
 	1000 1550 1000 1650
-Text Label 9700 2200 0    50   ~ 0
+Text Label 10150 2100 0    50   ~ 0
 SWDIO
-Text Label 9700 2300 0    50   ~ 0
+Text Label 10150 2300 0    50   ~ 0
 SWCLK
 $Comp
@@
 P 2700 4750
 F 0 "SW1" V 2654 4848 50  0000 L CNN
-F 1 "SW_SPST" V 2745 4848 50  0000 L CNN
+F 1 "~RST~" V 2745 4848 50  0000 L CNN
 F 2 "Button_Switch_SMD:SW_SPST_B3U-1000P" H 2700 4750 50  0001 C CNN
 F 3 "~" H 2700 4750 50  0001 C CNN
@@
 Text Label 1000 1950 0    50   ~ 0
 -
-$Comp
-L Connector:TestPoint TP101
-U 1 1 5E38CEFE
-P 10250 2200
-F 0 "TP101" V 10055 2272 50  0000 C CNN
-F 1 "SWDIO" V 10146 2272 50  0000 C CNN
-F 2 "TestPoint:TestPoint_Pad_D1.0mm" H 10450 2200 50  0001 C CNN
-F 3 "~" H 10450 2200 50  0001 C CNN
-	1    10250 2200
-	0    1    1    0
-$EndComp
-$Comp
-L Connector:TestPoint TP102
-U 1 1 5E38D660
-P 10250 2300
-F 0 "TP102" V 10204 2488 50  0000 L CNN
-F 1 "SWCLK" V 10295 2488 50  0000 L CNN
-F 2 "TestPoint:TestPoint_Pad_D1.0mm" H 10450 2300 50  0001 C CNN
-F 3 "~" H 10450 2300 50  0001 C CNN
-	1    10250 2300
-	0    1    1    0
-$EndComp
-Wire Wire Line
-	10250 2200 9500 2200
+Wire Wire Line
+	10700 2100 9950 2100
 Text Label 2500 2400 1    50   ~ 0
 PAVDD
@@
 NoConn ~ 3650 2900
 NoConn ~ 3650 3000
+$Comp
+L Connector_Generic:Conn_01x04 J1
+U 1 1 5E470F09
+P 10900 2200
+F 0 "J1" H 10980 2192 50  0000 L CNN
+F 1 "Conn_01x04" H 10980 2101 50  0000 L CNN
+F 2 "Connector_PinHeader_1.27mm:PinHeader_1x04_P1.27mm_Vertical" H 10900 2200 50  0001 C CNN
+F 3 "~" H 10900 2200 50  0001 C CNN
+	1    10900 2200
+	1    0    0    -1
+$EndComp
+$Comp
+L power:GND #PWR019
+U 1 1 5E47862B
+P 9950 2200
+F 0 "#PWR019" H 9950 1950 50  0001 C CNN
+F 1 "GND" V 9955 2072 50  0000 R CNN
+F 2 "" H 9950 2200 50  0001 C CNN
+F 3 "" H 9950 2200 50  0001 C CNN
+	1    9950 2200
+	0    1    1    0
+$EndComp
+Wire Wire Line
+	10700 2200 9950 2200
+$Comp
+L power:VDD #PWR020
+U 1 1 5E47C814
+P 9950 2400
+F 0 "#PWR020" H 9950 2250 50  0001 C CNN
+F 1 "VDD" V 9968 2527 50  0000 L CNN
+F 2 "" H 9950 2400 50  0001 C CNN
+F 3 "" H 9950 2400 50  0001 C CNN
+	1    9950 2400
+	0    -1   -1   0
+$EndComp
+Wire Wire Line
+	10700 2400 9950 2400
+$Comp
+L Switch:SW_SPST SW2
+U 1 1 5E492791
+P 1400 3450
+F 0 "SW2" V 1354 3548 50  0000 L CNN
+F 1 "USR" V 1445 3548 50  0000 L CNN
+F 2 "Button_Switch_SMD:SW_SPST_B3U-1000P" H 1400 3450 50  0001 C CNN
+F 3 "~" H 1400 3450 50  0001 C CNN
+	1    1400 3450
+	-1   0    0    1
+$EndComp
+Wire Wire Line
+	2150 3450 1600 3450
+Wire Wire Line
+	1200 3450 1100 3450
+$Comp
+L power:GND #PWR0102
+U 1 1 5E4A238D
+P 1100 3550
+F 0 "#PWR0102" H 1100 3300 50  0001 C CNN
+F 1 "GND" H 1105 3377 50  0000 C CNN
+F 2 "" H 1100 3550 50  0001 C CNN
+F 3 "" H 1100 3550 50  0001 C CNN
+	1    1100 3550
+	1    0    0    -1
+$EndComp
+Wire Wire Line
+	1100 3450 1100 3550
+Text Label 1700 3450 0    50   ~ 0
+~USRBTN~
 $EndSCHEMATC

Commit message: Fun tests
Changed lines of the file:
@@
 	1750 3250 2150 3250
 Wire Wire Line
-	1750 3350 2150 3350
+	3650 2800 4050 2800
 Text Label 1800 3150 0    50   ~ 0
 HDC_SDA
-Text Label 1800 3350 0    50   ~ 0
+Text Label 3750 2800 0    50   ~ 0
 HDC_INT
 Text Label 1800 3250 0    50   ~ 0
@@
 	2450 1250 2450 1300
 Connection ~ 2450 1250
-NoConn ~ 3650 2800
+NoConn ~ 2150 3350
 NoConn ~ 3650 2900
 NoConn ~ 3650 3000
