File: ilulissat.sch (KiCad schematic (older format))
At the start: 31 parts, among them J1 Conn_01x06, SW1 ~RST~, SW2 USR, U1 EFR32MG21x, U2 HDC2080, Y1 32.768Khz, Y2 38.4Mhz

Commit message: Rev1
Changed lines of the file:
@@
 U 1 1 5E3661FE
 P 2700 4750
-F 0 "SW1" V 2654 4848 50  0000 L CNN
-F 1 "~RST~" V 2745 4848 50  0000 L CNN
+F 0 "SW1" V 2600 4500 50  0000 L CNN
+F 1 "~RST~" V 2850 4550 50  0000 L CNN
 F 2 "Button_Switch_SMD:SW_SPST_B3U-1000P" H 2700 4750 50  0001 C CNN
 F 3 "~" H 2700 4750 50  0001 C CNN
